File: Kicad/FalloutTimer.kicad_sch (KiCad schematic)
At the start: 9 parts, among them J1 Conn_01x04_Pin, J2 Conn_01x04_Pin, J3 Conn_01x04_Pin, J4 Conn_01x04_Pin, J5 Conn_01x04_Pin, J6 Conn_01x04_Pin, J7 Conn_01x04_Pin, J8 Conn_01x04_Pin

Commit message: PCB and Schema mostly done
Parts:
- removed J1, J2, J3, J4, J5, J6, J7, J8: Conn_01x04_Pin, symbol Connector:Conn_01x04_Pin
- added C1: 100nF, Capacitor_THT:C_Disc_D5.0mm_W2.5mm_P5.00mm, symbol Device:C
- added J1: Conn_01x05_Pin, Connector_PinHeader_2.54mm:PinHeader_1x05_P2.54mm_Vertical, symbol Connector:Conn_01x05_Pin
- added SW1, SW2: SW_Push, Button_Switch_THT:SW_PUSH_6mm, symbol Switch:SW_Push
- added U1: DS3231M, Package_SO:SOIC-16W_7.5x10.3mm_P1.27mm, symbol Timer_RTC:DS3231M
Connections:
- net SCK: now reaches A1.1 (GPIO0)
- net SCK: now also J1.4 (Pin_4)
- net GND: now reaches A1.13 (GND), A1.18 (GND), A1.23 (GND), A1.28 (GND), A1.3 (GND), A1.38 (GND), A1.8 (GND)
- net GND: now also A1.33 (AGND), C1.2, J1.2 (Pin_2), SW1.2, SW2.2, U1.10 (GND), U1.11 (GND), U1.12 (GND), U1.13 (GND), U1.5 (GND), U1.6 (GND), U1.7 (GND), U1.8 (GND), U1.9 (GND)
- net DIO: now reaches A1.2 (GPIO1)
- net DIO: now also J1.5 (Pin_5)
- net SW1: now reaches A1.21 (GPIO16)
- net SW1: now also SW1.1
- net SW2: now reaches A1.22 (GPIO17)
- net SW2: now also SW2.1
- net SDA: now reaches A1.24 (GPIO18)
- net SDA: now also U1.15 (SDA)
- net SCL: now reaches A1.25 (GPIO19)
- net SCL: now also U1.16 (SCL)
- net 3.3v: now reaches A1.36 (3V3)
- net 3.3v: now also U1.2 (VCC)
- net RCK: now reaches A1.4 (GPIO2)
- net RCK: now also J1.3 (Pin_3)
- net +5V: now reaches A1.40 (VBUS)
- net +5V: now also C1.1, J1.1 (Pin_1)
- no-connect marks 0 -> 26
Other:
- note added: "Connect to 7 segment display"
- note removed: "Uhh put 8 7 segment displaus here laterrr"
